File: led-strip-controller.sch (KiCad schematic (older format))
At the start: 15 parts, among them CON1 BARREL_JACK, IC1 ATMEGA168-P, P2 CONN_01X04, U1 LM7805

Commit message: Update schematics a bit
Parts:
- added Q1, Q2, Q3: IRF640N, TO220, symbol IRF640N
Changed lines of the file:
@@
 $EndComp
 $Comp
-L VCC #PWR01
+L VCC #PWR5
 U 1 1 549C157A
 P 2300 1150
-F 0 "#PWR01" H 2300 1000 60  0001 C CNN
+F 0 "#PWR5" H 2300 1000 60  0001 C CNN
 F 1 "VCC" H 2300 1300 60  0000 C CNN
 F 2 "" H 2300 1150 60  0000 C CNN
@@
 $EndComp
 $Comp
-L GND #PWR02
+L GND #PWR6
 U 1 1 549C1625
 P 2450 1400
-F 0 "#PWR02" H 2450 1150 60  0001 C CNN
+F 0 "#PWR6" H 2450 1150 60  0001 C CNN
 F 1 "GND" H 2450 1250 60  0000 C CNN
 F 2 "" H 2450 1400 60  0000 C CNN
@@
 $EndComp
 $Comp
-L GND #PWR03
+L GND #PWR8
 U 1 1 549C1972
 P 5500 2550
-F 0 "#PWR03" H 5500 2300 60  0001 C CNN
+F 0 "#PWR8" H 5500 2300 60  0001 C CNN
 F 1 "GND" H 5500 2400 60  0000 C CNN
 F 2 "" H 5500 2550 60  0000 C CNN
@@
 $EndComp
 $Comp
-L GND #PWR04
+L GND #PWR12
 U 1 1 549C1AF4
 P 5950 3800
-F 0 "#PWR04" H 5950 3550 60  0001 C CNN
+F 0 "#PWR12" H 5950 3550 60  0001 C CNN
 F 1 "GND" H 5950 3650 60  0000 C CNN
 F 2 "" H 5950 3800 60  0000 C CNN
@@
 $EndComp
 $Comp
-L GND #PWR05
+L GND #PWR18
 U 1 1 549C1BDC
 P 9450 2900
-F 0 "#PWR05" H 9450 2650 60  0001 C CNN
+F 0 "#PWR18" H 9450 2650 60  0001 C CNN
 F 1 "GND" H 9450 2750 60  0000 C CNN
 F 2 "" H 9450 2900 60  0000 C CNN
@@
 $EndComp
 $Comp
-L +5V #PWR06
+L +5V #PWR9
 U 1 1 549C1DB7
 P 5850 1300
-F 0 "#PWR06" H 5850 1150 60  0001 C CNN
+F 0 "#PWR9" H 5850 1150 60  0001 C CNN
 F 1 "+5V" H 5850 1440 60  0000 C CNN
 F 2 "" H 5850 1300 60  0000 C CNN
@@
 $EndComp
 $Comp
-L +5V #PWR07
+L +5V #PWR10
 U 1 1 549C1DE1
 P 5850 1600
-F 0 "#PWR07" H 5850 1450 60  0001 C CNN
+F 0 "#PWR10" H 5850 1450 60  0001 C CNN
 F 1 "+5V" H 5850 1740 60  0000 C CNN
 F 2 "" H 5850 1600 60  0000 C CNN
@@
 $EndComp
 $Comp
-L +5V #PWR08
+L +5V #PWR11
 U 1 1 549C1DF2
 P 5850 1900
-F 0 "#PWR08" H 5850 1750 60  0001 C CNN
+F 0 "#PWR11" H 5850 1750 60  0001 C CNN
 F 1 "+5V" H 5850 2040 60  0000 C CNN
 F 2 "" H 5850 1900 60  0000 C CNN
@@
 $EndComp
 $Comp
-L +5V #PWR09
+L +5V #PWR17
 U 1 1 549C1E27
 P 9450 2400
-F 0 "#PWR09" H 9450 2250 60  0001 C CNN
+F 0 "#PWR17" H 9450 2250 60  0001 C CNN
 F 1 "+5V" H 9450 2540 60  0000 C CNN
 F 2 "" H 9450 2400 60  0000 C CNN
@@
 $EndComp
 $Comp
-L GND #PWR010
+L GND #PWR2
 U 1 1 549C1FF6
 P 2150 2850
-F 0 "#PWR010" H 2150 2600 60  0001 C CNN
+F 0 "#PWR2" H 2150 2600 60  0001 C CNN
 F 1 "GND" H 2150 2700 60  0000 C CNN
 F 2 "" H 2150 2850 60  0000 C CNN
@@
 $EndComp
 $Comp
-L VCC #PWR011
+L VCC #PWR1
 U 1 1 549C205A
 P 1550 2450
-F 0 "#PWR011" H 1550 2300 60  0001 C CNN
+F 0 "#PWR1" H 1550 2300 60  0001 C CNN
 F 1 "VCC" H 1550 2600 60  0000 C CNN
 F 2 "" H 1550 2450 60  0000 C CNN
@@
 $EndComp
 $Comp
-L +5V #PWR012
+L +5V #PWR7
 U 1 1 549C2096
 P 2750 2450
-F 0 "#PWR012" H 2750 2300 60  0001 C CNN
+F 0 "#PWR7" H 2750 2300 60  0001 C CNN
 F 1 "+5V" H 2750 2590 60  0000 C CNN
 F 2 "" H 2750 2450 60  0000 C CNN
@@
 $EndComp
 $Comp
-L +5V #PWR013
+L +5V #PWR3
 U 1 1 549EB884
 P 2200 3400
-F 0 "#PWR013" H 2200 3250 60  0001 C CNN
+F 0 "#PWR3" H 2200 3250 60  0001 C CNN
 F 1 "+5V" H 2200 3540 60  0000 C CNN
 F 2 "" H 2200 3400 60  0000 C CNN
@@
 $EndComp
 $Comp
-L GND #PWR014
+L GND #PWR4
 U 1 1 549EB941
 P 2200 4450
-F 0 "#PWR014" H 2200 4200 60  0001 C CNN
+F 0 "#PWR4" H 2200 4200 60  0001 C CNN
 F 1 "GND" H 2200 4300 60  0000 C CNN
 F 2 "" H 2200 4450 60  0000 C CNN
@@
 	6650 4800 6650 4900
 $Comp
-L VCC #PWR018
+L VCC #PWR16
 U 1 1 54A21678
 P 9400 5350
-F 0 "#PWR018" H 9400 5200 60  0001 C CNN
+F 0 "#PWR16" H 9400 5200 60  0001 C CNN
 F 1 "VCC" H 9400 5500 60  0000 C CNN
 F 2 "" H 9400 5350 60  0000 C CNN
@@
 	8450 5650 8450 5800
 $Comp
-L GND #PWR?
+L GND #PWR13
 U 1 1 54AEB316
 P 7050 5800
-F 0 "#PWR?" H 7050 5550 60  0001 C CNN
+F 0 "#PWR13" H 7050 5550 60  0001 C CNN
 F 1 "GND" H 7050 5650 60  0000 C CNN
 F 2 "" H 7050 5800 60  0000 C CNN
@@
 $EndComp
 $Comp
-L GND #PWR?
+L GND #PWR14
 U 1 1 54AEB38E
 P 7750 5800
-F 0 "#PWR?" H 7750 5550 60  0001 C CNN
+F 0 "#PWR14" H 7750 5550 60  0001 C CNN
 F 1 "GND" H 7750 5650 60  0000 C CNN
 F 2 "" H 7750 5800 60  0000 C CNN
@@
 $EndComp
 $Comp
-L GND #PWR?
+L GND #PWR15
 U 1 1 54AEB3AB
 P 8450 5800
-F 0 "#PWR?" H 8450 5550 60  0001 C CNN
+F 0 "#PWR15" H 8450 5550 60  0001 C CNN
 F 1 "GND" H 8450 5650 60  0000 C CNN
 F 2 "" H 8450 5800 60  0000 C CNN
@@
 Text Label 7050 5150 0    60   ~ 0
 B
+$Comp
+L IRF640N Q1
+U 1 1 553395DC
+P 6950 5450
+F 0 "Q1" H 6950 5302 40  0000 R CNN
+F 1 "IRF640N" H 6950 5599 40  0000 R CNN
+F 2 "TO220" H 6771 5551 29  0000 C CNN
+F 3 "" H 6950 5450 60  0000 C CNN
+	1    6950 5450
+	1    0    0    -1
+$EndComp
+$Comp
+L IRF640N Q2
+U 1 1 55339A4B
+P 7650 5450
+F 0 "Q2" H 7650 5302 40  0000 R CNN
+F 1 "IRF640N" H 7650 5599 40  0000 R CNN
+F 2 "TO220" H 7471 5551 29  0000 C CNN
+F 3 "" H 7650 5450 60  0000 C CNN
+	1    7650 5450
+	1    0    0    -1
+$EndComp
+$Comp
+L IRF640N Q3
+U 1 1 55339A9F
+P 8350 5450
+F 0 "Q3" H 8350 5302 40  0000 R CNN
+F 1 "IRF640N" H 8350 5599 40  0000 R CNN
+F 2 "TO220" H 8171 5551 29  0000 C CNN
+F 3 "" H 8350 5450 60  0000 C CNN
+	1    8350 5450
+	1    0    0    -1
+$EndComp
 $EndSCHEMATC
